Commit message: rotate in urdf

File: src/abot_description/urdf/abot_caster_wheel.xacro (robot description, xacro)
@@ -24,5 +24,5 @@
 	</link>
 	<joint name="caster_wheel_to_base" type="continuous">
-		<origin xyz="-0.078 0 -0.011" rpy="0 0 0" />
+		<origin xyz="-0.078 0 -0.011" rpy="0 0 ${PI}" />
 		<parent link="abot_base" />
 		<child link="abot_caster_wheel" />

File: src/abot_description/urdf/abot_left_wheel.xacro (robot description, xacro)
@@ -45,5 +45,5 @@
 	</joint>
 	<joint name="left_wheel_to_base" type="continuous">
-		<origin xyz="0 0.068 0.0145" rpy="0 0 0" />
+		<origin xyz="0 0.068 0.0145" rpy="0 0 ${PI}" />
 		<parent link="abot_base" />
 		<child link="left_wheel" />

File: src/abot_description/urdf/abot_right_wheel.xacro (robot description, xacro)
@@ -45,5 +45,5 @@
 	</joint>
 	<joint name="right_wheel_to_base" type="continuous">
-		<origin xyz="0 -0.068 0.0145" rpy="0 0 0" />
+		<origin xyz="0 -0.068 0.0145" rpy="0 0 ${PI}" />
 		<parent link="abot_base" />
 		<child link="right_wheel" />
